File: 65-o-clock.kicad_pcb (KiCad board)
At the start: 2 copper layers, 161.3 x 161.3 mm, 103 parts, among them J1 USB_B_Micro, SW1 SW_Push, SW2 SW_Push, SW3 SW_Push, U1 W65C02, U10 KCSC02-107, U11 KCSC02-107, U12 KCSC02-107, U13 KCSC02-107, U2 7400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

Commit message: Diodes placed, layout started
Parts:
- moved X1 255.6 mm to (105.4, 96.5), turned to 270 degrees
- moved U1 216.0 mm to (120.7, 95.2)
- moved U8 214.2 mm to (105.4, 58.4)
- moved U4 206.1 mm to (158.1, 149.9), turned to 180 degrees
- moved U2 205.0 mm to (193.7, 132.1), turned to 180 degrees
- moved U3 202.7 mm to (181.0, 149.9), turned to 180 degrees
- moved U9 201.3 mm to (116.2, 58.4)
- moved U6 152.9 mm to (191.1, 58.3)
- moved U7 130.3 mm to (202.6, 58.3)
- moved U5 126.1 mm to (191.1, 95.2), turned to 270 degrees
- turned D10 to 210 degrees
- turned D11 to 204 degrees
- turned D12 to 198 degrees
- turned D13 to 192 degrees
- turned D14 to 186 degrees
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Routing:
- net Net-(D10-Pad1): track 0.00 -> 55.1 mm
- net Net-(D17-Pad1): track 0.00 -> 55.0 mm
- net Net-(D33-Pad1): track 0.00 -> 55.0 mm
- net Net-(D1-Pad1): track 0.00 -> 55.0 mm
- net Net-(D49-Pad1): track 0.00 -> 55.0 mm
- net Net-(D41-Pad1): track 0.00 -> 55.0 mm
- net Net-(D25-Pad1): track 0.00 -> 55.0 mm
- net /A3: track 0.00 -> 49.6 mm, vias 0 -> 1
- net /A2: track 0.00 -> 47.6 mm, vias 0 -> 1
- net /A1: track 0.00 -> 46.0 mm, vias 0 -> 1
- net /A0: track 0.00 -> 44.3 mm, vias 0 -> 1
- net /D7: track 0.00 -> 39.7 mm, vias 0 -> 1
- net /D6: track 0.00 -> 37.7 mm, vias 0 -> 1
- net /D0: track 0.00 -> 36.6 mm, vias 0 -> 1
- net /D5: track 0.00 -> 34.7 mm, vias 0 -> 1
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